File: shield.sch (KiCad schematic (older format))
At the start: 17 parts

Commit message: pin assignment, separate CAN_5V
Parts:
- removed P?: Servo_5V, symbol CONN_01X02
- removed P?: CAN_5V, symbol CONN_01X02
- added CONN?: SWD/DEBUG, MODULE, symbol SWD/DEBUG
Connections:
- net +5V: now also P?.1 (P1), CONN?.1 (VCC)
- net ENCODER_LEFT_CHA: now also P?.3 (P3), U?.43B (PD12)
- net ENCODER_LEFT_CHB: now also P?.4 (P4), U?.41B (PD13)
- net ENCODER_LEFT_CHI: now also P?.5 (P5), U?.45B (PD11)
- net ENCODER_RIGHT_CHA: now also P?.3 (P3), U?.4B (PC6)
- net ENCODER_RIGHT_CHB: now also P?.4 (P4), U?.19B (PC7)
- net ENCODER_RIGHT_CHI: now also P?.5 (P5), U?.26B (PB15)
- net ENCODER_TRANSVERS_CHA: now also P?.3 (P3), U?.50A (PE5)
- net ENCODER_TRANSVERS_CHB: now also P?.4 (P4), U?.62A (PE6)
- net ENCODER_TRANSVERS_CHI: now also P?.5 (P5), U?.48A (PE4)
- net GND: now also P?.2 (P2), CONN?.2 (GND), CONN?.MECH (GND)
- net SWDIO: now reaches U?.13A (PA13)
- net SWDIO: now also CONN?.4 (SWDIO)
- net NRST: now reaches U?.14A (RESET)
- net NRST: now also CONN?.3 (NRST)
- net SWCLK: now reaches U?.15A (PA14)
- net SWCLK: now also CONN?.5 (SWCLK)
- net DEBUG_UART_RX: now reaches U?.69A (PD9)
- net DEBUG_UART_RX: now also CONN?.7 (RX)
- net DEBUG_UART_TX: now reaches U?.10B (PD8)
- net DEBUG_UART_TX: now also CONN?.6 (TX)
- net CAN1L: now reaches P?.17 (P17)
- net CAN1H: now reaches P?.18 (P18)
- net CAN2L: now reaches P?.19 (P19)
- net CAN2H: now reaches P?.20 (P20)
- no-connect marks 0 -> 1
Other:
- moved on the sheet: U?B
Changed lines of the file:
@@
 L ST_Nucleo144_F429ZI_Morpho U?
 U 2 1 57E00191
-P 4450 2850
-F 0 "U?" H 4200 4700 60  0000 C CNN
-F 1 "ST_Nucleo144_F429ZI_Morpho" V 4450 2850 60  0000 C CNN
-F 2 "" H 4450 3200 60  0000 C CNN
-F 3 "" H 4450 3200 60  0000 C CNN
-	2    4450 2850
+P 5250 2850
+F 0 "U?" H 5000 4700 60  0000 C CNN
+F 1 "ST_Nucleo144_F429ZI_Morpho" V 5250 2850 60  0000 C CNN
+F 2 "" H 5250 3200 60  0000 C CNN
+F 3 "" H 5250 3200 60  0000 C CNN
+	2    5250 2850
 	1    0    0    -1
 $EndComp
@@
 GPIO4
 $Sheet
-S 9900 5650 1100 650
+S 9550 5650 1100 650
 U 58172972
 F0 "CAN interfaces" 60
 F1 "can_interfaces.sch" 60
-F2 "CAN1_RX" I L 9900 5750 60
-F3 "CAN1_TX" O L 9900 5850 60
-F4 "CAN2_RX" I L 9900 6050 60
-F5 "CAN2_TX" O L 9900 6150 60
-F6 "CAN1H" B R 11000 5750 60
-F7 "CAN1L" B R 11000 5850 60
-F8 "CAN2H" B R 11000 6050 60
-F9 "CAN2L" B R 11000 6150 60
+F2 "CAN1_RX" I L 9550 5750 60
+F3 "CAN1_TX" O L 9550 5850 60
+F4 "CAN2_RX" I L 9550 6050 60
+F5 "CAN2_TX" O L 9550 6150 60
+F6 "CAN1H" B R 10650 5750 60
+F7 "CAN1L" B R 10650 5850 60
+F8 "CAN2H" B R 10650 6050 60
+F9 "CAN2L" B R 10650 6150 60
 $EndSheet
-$Comp
-L CONN_01X02 P?
-U 1 1 58173DDD
-P 10900 4100
-F 0 "P?" H 10900 4250 50  0000 C CNN
-F 1 "Servo_5V" V 11000 4100 50  0000 C CNN
-F 2 "" H 10900 4100 50  0000 C CNN
-F 3 "" H 10900 4100 50  0000 C CNN
-	1    10900 4100
-	1    0    0    -1
-$EndComp
-$Comp
-L CONN_01X02 P?
-U 1 1 58173F03
-P 10900 4500
-F 0 "P?" H 10900 4650 50  0000 C CNN
-F 1 "CAN_5V" V 11000 4500 50  0000 C CNN
-F 2 "" H 10900 4500 50  0000 C CNN
-F 3 "" H 10900 4500 50  0000 C CNN
-	1    10900 4500
-	1    0    0    -1
-$EndComp
 $Comp
 L MICRO_SD CONN?
@@
 Text Label 1950 7050 2    50   ~ 0
 SDIO_CK
-Text Label 3800 1250 2    50   ~ 0
+Text Label 4600 1250 2    50   ~ 0
 SD_DETECT
 Text Label 2050 7650 0    50   ~ 0
@@
 Text Label 1400 1150 2    50   ~ 0
 SDIO_D2
-Text Label 3800 1150 2    50   ~ 0
+Text Label 4600 1150 2    50   ~ 0
 SDIO_D1
-Text Label 5100 1150 0    50   ~ 0
+Text Label 5900 1150 0    50   ~ 0
 SDIO_D0
 Text Label 2700 1250 0    50   ~ 0
@@
 Wire Wire Line
 	1350 6650 1350 6850
-Text Label 3800 1350 2    50   ~ 0
+Text Label 4600 1350 2    50   ~ 0
 SD_PWR
 $Comp
@@
 ENCODER_LEFT_CHI
 $Sheet
-S 8150 5650 1050 500
+S 7150 5650 1050 500
 U 584D3A1E
 F0 "servo" 60
 F1 "servo.sch" 60
-F2 "SERVO_I2C_SDA" B L 8150 5850 60
-F3 "SERVO_I2C_SCL" I L 8150 5950 60
-F4 "SERVO_OE" I L 8150 5750 60
+F2 "SERVO_I2C_SDA" B L 7150 5850 60
+F3 "SERVO_I2C_SCL" I L 7150 5950 60
+F4 "SERVO_OE" I L 7150 5750 60
 $EndSheet
-Text Label 9500 5850 0    50   ~ 0
+Text Label 9150 5850 0    50   ~ 0
 CAN1_TX
-Text Label 9500 5750 0    50   ~ 0
+Text Label 9150 5750 0    50   ~ 0
 CAN1_RX
 Text Label 1400 3950 2    50   ~ 0
 CAN1_RX
 Wire Wire Line
-	9500 5750 9900 5750
+	9150 5750 9550 5750
 Text Label 1400 3850 2    50   ~ 0
 CAN1_TX
 Wire Wire Line
-	9500 5850 9900 5850
-Text Label 3800 1950 2    50   ~ 0
+	9150 5850 9550 5850
+Text Label 4600 1950 2    50   ~ 0
 CAN2_TX
-Text Label 3800 2550 2    50   ~ 0
+Text Label 4600 2550 2    50   ~ 0
 CAN2_RX
-Text Label 9500 6050 0    50   ~ 0
+Text Label 9150 6050 0    50   ~ 0
 CAN2_RX
-Text Label 9500 6150 0    50   ~ 0
+Text Label 9150 6150 0    50   ~ 0
 CAN2_TX
 Wire Wire Line
-	9500 6150 9900 6150
-Wire Wire Line
-	9900 6050 9500 6050
+	9150 6150 9550 6150
+Wire Wire Line
+	9550 6050 9150 6050
 $Comp
 L CONN_01X05 P?
@@
 Text Label 6650 3400 0    50   ~ 0
 ENCODER_TRANSVERS_CHI
-Text Label 5100 3850 0    50   ~ 0
+Text Label 5900 3850 0    50   ~ 0
 SPI4_CS
-Text Label 3800 3550 2    50   ~ 0
+Text Label 4600 3550 2    50   ~ 0
 SPI4_SCK
-Text Label 3800 3850 2    50   ~ 0
+Text Label 4600 3850 2    50   ~ 0
 SPI4_MISO
-Text Label 3800 3650 2    50   ~ 0
+Text Label 4600 3650 2    50   ~ 0
 SPI4_MOSI
 Text Label 10550 2950 2    50   ~ 0
@@
 	1    0    0    -1
 $EndComp
-Text Label 3800 2350 2    50   ~ 0
+Text Label 4600 2350 2    50   ~ 0
 I2C2_SCL
-Text Label 5100 1950 0    50   ~ 0
+Text Label 5900 1950 0    50   ~ 0
 I2C2_SDA
 Text Label 1400 3150 2    50   ~ 0
@@
 	1    0    0    -1
 $EndComp
+$Comp
+L SWD/DEBUG CONN?
+U 1 1 585B6C63
+P 6200 6500
+F 0 "CONN?" H 6200 6950 50  0000 C CNN
+F 1 "SWD/DEBUG" H 6200 6050 50  0000 C CNN
+F 2 "MODULE" H 6200 6450 50  0001 C CNN
+F 3 "DOCUMENTATION" H 6200 6450 50  0001 C CNN
+	1    6200 6500
+	1    0    0    -1
+$EndComp
+Text Label 5900 1250 0    50   ~ 0
+ENCODER_RIGHT_CHA
+Text Label 4600 2050 2    50   ~ 0
+ENCODER_RIGHT_CHB
+Text Label 5900 2350 0    50   ~ 0
+ENCODER_RIGHT_CHI
+NoConn ~ 5900 1350
+Text Label 4600 3250 2    50   ~ 0
+ENCODER_LEFT_CHA
+Text Label 4600 3150 2    50   ~ 0
+ENCODER_LEFT_CHB
+Text Label 4600 3350 2    50   ~ 0
+ENCODER_LEFT_CHI
+Text Label 2700 3550 0    50   ~ 0
+ENCODER_TRANSVERS_CHA
+Text Label 2700 4150 0    50   ~ 0
+ENCODER_TRANSVERS_CHB
+Text Label 2700 3450 0    50   ~ 0
+ENCODER_TRANSVERS_CHI
+$Comp
+L +5V #PWR?
+U 1 1 586DB6CC
+P 7700 3000
+F 0 "#PWR?" H 7700 3090 20  0001 C CNN
+F 1 "+5V" H 7700 3090 30  0000 C CNN
+F 2 "" H 7700 3000 60  0000 C CNN
+F 3 "" H 7700 3000 60  0000 C CNN
+	1    7700 3000
+	1    0    0    -1
+$EndComp
+$Comp
+L GND #PWR?
+U 1 1 586DB74F
+P 7700 3100
+F 0 "#PWR?" H 7700 3100 30  0001 C CNN
+F 1 "GND" H 7700 3030 30  0001 C CNN
+F 2 "" H 7700 3100 60  0000 C CNN
+F 3 "" H 7700 3100 60  0000 C CNN
+	1    7700 3100
+	1    0    0    -1
+$EndComp
+Wire Wire Line
+	7700 3200 6650 3200
+Wire Wire Line
+	6650 3300 7700 3300
+Wire Wire Line
+	6650 3400 7700 3400
+Wire Wire Line
+	6850 3950 7700 3950
+Wire Wire Line
+	6850 4050 7700 4050
+Wire Wire Line
+	6850 4150 7700 4150
+Wire Wire Line
+	6850 4600 7700 4600
+Wire Wire Line
+	6850 4700 7700 4700
+Wire Wire Line
+	7700 4800 6850 4800
+Text Label 5850 6700 2    50   ~ 0
+DEBUG_UART_TX
+Text Label 5850 6800 2    50   ~ 0
+DEBUG_UART_RX
+Text Label 1400 4550 2    50   ~ 0
+DEBUG_UART_RX
+Text Label 5900 1550 0    50   ~ 0
+DEBUG_UART_TX
+Text Label 5850 6600 2    50   ~ 0
+SWCLK
+Text Label 5850 6500 2    50   ~ 0
+SWDIO
+Text Label 5850 6400 2    50   ~ 0
+NRST
+$Comp
+L GND #PWR?
+U 1 1 586DD8E9
+P 5850 6300
+F 0 "#PWR?" H 5850 6300 30  0001 C CNN
+F 1 "GND" H 5850 6230 30  0001 C CNN
+F 2 "" H 5850 6300 60  0000 C CNN
+F 3 "" H 5850 6300 60  0000 C CNN
+	1    5850 6300
+	1    0    0    -1
+$EndComp
+$Comp
+L +5V #PWR?
+U 1 1 586DD9D9
+P 5850 6200
+F 0 "#PWR?" H 5850 6290 20  0001 C CNN
+F 1 "+5V" H 5850 6290 30  0000 C CNN
+F 2 "" H 5850 6200 60  0000 C CNN
+F 3 "" H 5850 6200 60  0000 C CNN
+	1    5850 6200
+	1    0    0    -1
+$EndComp
+Text Label 2700 1750 0    50   ~ 0
+NRST
+Text Label 1400 1750 2    50   ~ 0
+SWDIO
+Text Label 1400 1850 2    50   ~ 0
+SWCLK
+Text Label 10950 5750 2    50   ~ 0
+CAN1H
+Text Label 10950 6050 2    50   ~ 0
+CAN2H
+Text Label 10950 5850 2    50   ~ 0
+CAN1L
+Text Label 10950 6150 2    50   ~ 0
+CAN2L
+Wire Wire Line
+	10650 6050 10950 6050
+Wire Wire Line
+	10650 6150 10950 6150
+Wire Wire Line
+	10650 5850 10950 5850
+Wire Wire Line
+	10650 5750 10950 5750
+Text Label 9700 1600 0    50   ~ 0
+CAN1H
+Text Label 9200 1600 2    50   ~ 0
+CAN1L
+Text Label 9700 1700 0    50   ~ 0
+CAN2H
+Text Label 9200 1700 2    50   ~ 0
+CAN2L
 $EndSCHEMATC

Commit message: pin assignment, symbol placement
Parts:
- added P?: CONN_01X03, symbol CONN_01X03
- added R? (x4): 4.7k, symbol R
Connections:
- net ENCODER_RIGHT_CHI: no longer U?.26B (PB15)
- net GND: now also P?.3 (P3)
- net GPIO1: now also U?.63A (PG9)
- net GPIO2: now also U?.61B (PG14)
- net GPIO3: now also U?.64A (PG15)
- net GPIO4: now also U?.65A (PG12)
- net I2C2_SCL: now also R?.2
- net I2C2_SDA: now also R?.2
- net SD_DETECT: now also U?.11B (PA5); no longer U?.3B (PB8)
- net SD_PWR: now also U?.13B (PA6); no longer U?.5B (PB9)
- net VCC: now also P?.1 (P1), R?.1, R?.1, R?.1, R?.1
- net EXT_IO_7: now reaches U?.11A (PF7)
- net EXT_IO_7: now also P?.10 (P10)
- net SERVO_OE: now reaches U?.38A (PC0)
- net EXT_IO_1: now reaches U?.51A (PF1)
- net EXT_IO_1: now also P?.4 (P4)
- net EXT_IO_2: now reaches U?.52A (PF2)
- net EXT_IO_2: now also P?.5 (P5)
- net EXT_IO_0: now reaches U?.53A (PF0)
- net EXT_IO_0: now also P?.3 (P3)
- net EXT_IO_8: now reaches U?.54A (PF8)
- net EXT_IO_8: now also P?.11 (P11)
- net EXT_IO_9: now reaches U?.56A (PF9)
- net EXT_IO_9: now also P?.12 (P12)
- net EXT_IO_6: now reaches U?.9A (PF6)
- net EXT_IO_6: now also P?.9 (P9)
- net ROBOT_SELECT: now reaches U?.24B (PB1)
- net ROBOT_SELECT: now also P?.2 (P2)
- net EXT_IO_5: now reaches U?.36B (PF5)
- net EXT_IO_5: now also P?.8 (P8)
- net EXT_IO_4: now reaches U?.38B (PF4)
- net EXT_IO_4: now also P?.7 (P7)
- net EXT_IO_10: now reaches U?.42B (PF10)
- net EXT_IO_10: now also P?.13 (P13)
- net LED_RGB_B: now reaches U?.57B (PF13)
- net LED_RGB_B: now also P?.16 (P16)
- net EXT_IO_3: now reaches U?.58B (PF3)
- net EXT_IO_3: now also P?.6 (P6)
- net LED_RGB_G: now reaches U?.59B (PF12)
- net LED_RGB_G: now also P?.15 (P15)
- net LED_RGB_R: now reaches U?.62B (PF11)
- net LED_RGB_R: now also P?.14 (P14)
- new net I2C1_SCL: R?.2, U?.3B (PB8)
- new net I2C1_SDA: R?.2, U?.5B (PB9)
- no-connect marks 1 -> 2
Other:
- note added: "BOOT1"
- note added: "Select robot\nbig robot = VCC\nsmall robot = GND"
- moved on the sheet: C?, CONN?, P?, Q?, R?, U?B

Commit message: footprint assignment
Parts:
- added J1: E5V_Conn, Terminal_Blocks:TerminalBlock_Pheonix_MKDS1.5-2pol, symbol Screw_Terminal_1x02
- added P6: 5V_CAN_SELECT, Pin_Headers:Pin_Header_Straight_2x02, symbol CONN_02X02
- C1: renamed from C?; value C -> 10uF; footprint (none) -> Capacitors_SMD:C_0805
- C2: renamed from C?; value C -> 100nF; footprint (none) -> Capacitors_SMD:C_0603
- CONN1: renamed from CONN?; footprint MODULE -> _div:_Molex-microSD-502570-0893
- CONN2: renamed from CONN?; footprint MODULE -> _connectors:_Molex-PicoBlade-SMD-7
- CONN3, CONN4: renamed from CONN?; footprint MODULE -> _connectors:Molex-PicoBlade-4
- CONN5: renamed from CONN?; footprint (none) -> _connectors:Molex-PicoBlade-6
- P1: renamed from P?; footprint (none) -> Pin_Headers:Pin_Header_Straight_1x03
- P2: renamed from P?; footprint (none) -> Pin_Headers:Pin_Header_Straight_2x10
- P3, P4, P5: renamed from P?; footprint (none) -> _connectors:Molex-PicoBlade-5
- P7: renamed from P?; footprint (none) -> Pin_Headers:Pin_Header_Straight_2x05
- Q1: renamed from Q?; footprint (none) -> TO_SOT_Packages_SMD:SOT-23_Handsoldering
- R1: renamed from R?; value R -> 10k; footprint (none) -> Resistors_SMD:R_0603
- R2, R3, R4, R5: renamed from R?; footprint (none) -> Resistors_SMD:R_0603
- U1: renamed from U?; footprint (none) -> _connectors:ST_Nucleo144_F429ZI_Morpho
Connections:
- net VCC is gone; now on net +3.3V: CONN3.1 (VCC), CONN4.1 (VCC), CONN5.1 (VCC), P1.1 (P1), Q1.1 (D), R1.1, R2.1, R3.1, R4.1, R5.1
- net +5V: now also U1.18A (+5V)
- net ENCODER_RIGHT_CHI: now also U1.26B (PB15)
- net GND: now also U1.19A (GND), U1.20A (GND), U1.20B (GND), U1.22A (GND), U1.32B (AGND), U1.39B (GND), U1.49A (GND), U1.54B (GND), U1.60A (GND), U1.63B (GND), U1.8A (GND), U1.9B (GND), J1.1
- net +3.3V: now reaches U1.16A (+3V3)
- net E5V: now reaches U1.6A (E5V)
- net E5V: now also J1.2, P6.1 (P1), P6.3 (P3)
- new net CAN interfaces/5V_CAN1: P6.2 (P2)
- new net CAN interfaces/5V_CAN2: P6.4 (P4)
Other:
- note added: "(BOOT1)"
- note added: "(select E5V with JP3 on Nucleo)"
- note added: "Extension connectors\nnot populated"
- note added: "Select robot:\nbig robot = VCC\nsmall robot = GND"
- note removed: "BOOT1"
- note removed: "Select robot\nbig robot = VCC\nsmall robot = GND"
- moved on the sheet: C1, CONN2, P1, P2, P3, P4, P5, P7
