File: shield.sch (KiCad schematic (older format))
At the start: 24 parts, among them J1 E5V_Conn, P1 ROBOT SELECT, P2 CONN_02X10, P3 ENCODER_TRANS, P4 ENCODER_RIGHT, P5 ENCODER_LEFT, P6 5V_CAN_SELECT, P7 GPIO, Q1 Q_PMOS_DGS, U1 ST_Nucleo144_F429ZI_Morpho

Commit message: PCB routing
Parts:
- added R8: 100, Resistors_SMD:R_0805, symbol R
- CONN2: footprint Connectors_Molex:Molex_PicoBlade_53047-0710_07x1.25mm_Straight -> Connectors_Molex:Molex_PicoBlade_53261-0771_07x1.25mm_Angled
- P7: footprint Connect:IDC_Header_Straight_10pins -> Pin_Headers:Pin_Header_Straight_2x05
Connections:
- net DEBUG_UART_RX: now also U1.9A (PF6); no longer U1.69A (PD9)
- net DEBUG_UART_TX: now also U1.11A (PF7); no longer U1.10B (PD8)
- net E5V: now also J1.1; no longer J1.2
- net EXT_IO_0: now also U1.61A (PE1); no longer U1.53A (PF0)
- net EXT_IO_1: now also U1.59A (PG0); no longer U1.51A (PF1)
- net EXT_IO_10: now also U1.66B (PG8); no longer U1.42B (PF10)
- net EXT_IO_2: now also U1.69A (PD9); no longer U1.52A (PF2)
- net EXT_IO_3: now also U1.66A (PG10); no longer U1.58B (PF3)
- net EXT_IO_4: now also U1.58A (PG1); no longer U1.38B (PF4)
- net EXT_IO_5: now also U1.56A (PF9); no longer U1.36B (PF5)
- net EXT_IO_6: now also U1.69B (PG4); no longer U1.9A (PF6)
- net EXT_IO_7: now also U1.65B (PD10); no longer U1.11A (PF7)
- net EXT_IO_8: now also U1.68B (PG5); no longer U1.54A (PF8)
- net EXT_IO_9: now also U1.64B (PE0); no longer U1.56A (PF9)
- net GND: now also J1.2; no longer J1.1
- net LED_SD: now also U1.16B (PB12)
- net SWDIO: now also R8.2; no longer CONN2.4 (SWDIO)
- new net: CONN2.4 (SWDIO), R8.1
- no-connect marks 2 -> 8
Changed lines of the file:
@@
 F 0 "P7" H 9500 5150 50  0000 C CNN
 F 1 "GPIO" H 9500 4550 50  0000 C CNN
-F 2 "Connect:IDC_Header_Straight_10pins" H 9500 3650 50  0001 C CNN
+F 2 "Pin_Headers:Pin_Header_Straight_2x05" H 9500 3650 50  0001 C CNN
 F 3 "" H 9500 3650 50  0000 C CNN
 	1    9500 4850
@@
 F 0 "CONN2" H 5550 7350 50  0000 C CNN
 F 1 "SWD/DEBUG" H 5550 6450 50  0000 C CNN
-F 2 "Connectors_Molex:Molex_PicoBlade_53047-0710_07x1.25mm_Straight" H 5550 6850 50  0001 C CNN
+F 2 "Connectors_Molex:Molex_PicoBlade_53261-0771_07x1.25mm_Angled" H 5550 6850 50  0001 C CNN
 F 3 "DOCUMENTATION" H 5550 6850 50  0001 C CNN
 	1    5550 6900
@@
 Text Label 5200 7200 2    50   ~ 0
 DEBUG_UART_RX
-Text Label 1400 4550 2    50   ~ 0
+Text Label 1400 1550 2    50   ~ 0
 DEBUG_UART_RX
-Text Label 6000 1550 0    50   ~ 0
+Text Label 1400 1650 2    50   ~ 0
 DEBUG_UART_TX
 Text Label 5200 7000 2    50   ~ 0
 SWCLK
-Text Label 5200 6900 2    50   ~ 0
+Text Label 4550 6900 2    50   ~ 0
 SWDIO
 Text Label 5200 6800 2    50   ~ 0
@@
 Text Label 7450 3700 2    50   ~ 0
 LED_RGB_G
-Text Label 1400 3750 2    50   ~ 0
+Text Label 1400 4150 2    50   ~ 0
 EXT_IO_0
-Text Label 1400 3650 2    50   ~ 0
+Text Label 1400 4050 2    50   ~ 0
 EXT_IO_1
-Text Label 2700 3650 0    50   ~ 0
+Text Label 1400 4550 2    50   ~ 0
 EXT_IO_2
-Text Label 6000 2950 0    50   ~ 0
+Text Label 2700 3950 0    50   ~ 0
 EXT_IO_4
-Text Label 1400 1550 2    50   ~ 0
+Text Label 4700 4550 2    50   ~ 0
 EXT_IO_6
-Text Label 2700 3750 0    50   ~ 0
+Text Label 6000 4450 0    50   ~ 0
 EXT_IO_8
-Text Label 6000 3150 0    50   ~ 0
+Text Label 6000 4350 0    50   ~ 0
 EXT_IO_10
 Text Label 4700 4050 2    50   ~ 0
 LED_RGB_G
-Text Label 6000 3950 0    50   ~ 0
+Text Label 2700 4350 0    50   ~ 0
 EXT_IO_3
-Text Label 6000 2850 0    50   ~ 0
+Text Label 2700 3850 0    50   ~ 0
 EXT_IO_5
-Text Label 1400 1650 2    50   ~ 0
+Text Label 4700 4350 2    50   ~ 0
 EXT_IO_7
-Text Label 2700 3850 0    50   ~ 0
+Text Label 6000 4250 0    50   ~ 0
 EXT_IO_9
 Text Label 6000 4150 0    50   ~ 0
@@
 Text Label 2700 1350 0    50   ~ 0
 E5V
-Text Label 8250 1950 0    50   ~ 0
+Text Label 8250 2150 0    50   ~ 0
 E5V
 $Comp
 L GND #PWR019
 U 1 1 58BB229F
-P 8700 2150
-F 0 "#PWR019" H 8700 2150 30  0001 C CNN
-F 1 "GND" H 8700 2080 30  0001 C CNN
-F 2 "" H 8700 2150 60  0001 C CNN
-F 3 "" H 8700 2150 60  0001 C CNN
-	1    8700 2150
+P 8700 1950
+F 0 "#PWR019" H 8700 1950 30  0001 C CNN
+F 1 "GND" H 8700 1880 30  0001 C CNN
+F 2 "" H 8700 1950 60  0001 C CNN
+F 3 "" H 8700 1950 60  0001 C CNN
+	1    8700 1950
 	1    0    0    -1
 $EndComp
@@
 	9600 2700 9150 2700
 Wire Wire Line
-	8250 1950 8700 1950
-Wire Wire Line
-	8500 1950 8500 2600
+	8250 2150 8700 2150
+Wire Wire Line
+	8500 2150 8500 2600
 Wire Wire Line
 	8500 2600 8650 2600
-Connection ~ 8500 1950
+Connection ~ 8500 2150
 Wire Wire Line
 	8650 2600 8650 2700
@@
 	0    -1   -1   0
 $EndComp
+$Comp
+L R R8
+U 1 1 58BC787B
+P 4800 6900
+F 0 "R8" V 4880 6900 50  0000 C CNN
+F 1 "100" V 4800 6900 50  0000 C CNN
+F 2 "Resistors_SMD:R_0805" V 4730 6900 50  0001 C CNN
+F 3 "" H 4800 6900 50  0000 C CNN
+	1    4800 6900
+	0    1    1    0
+$EndComp
+Wire Wire Line
+	4650 6900 4550 6900
+Wire Wire Line
+	4950 6900 5200 6900
+Text Label 6000 1850 0    50   ~ 0
+LED_SD
+NoConn ~ 6000 4550
+NoConn ~ 4700 4450
+NoConn ~ 2700 4450
+NoConn ~ 2700 4550
+NoConn ~ 4700 2150
+NoConn ~ 4700 2250
 $EndSCHEMATC

Commit message: change some GPIOs, finish routing
Parts:
- R8: value 100 -> 0
Connections:
- net +3.3V: now also CONN2.1 (VCC)
- net +5V: no longer CONN2.1 (VCC)
- net EXT_IO_6: now also U1.60B (PF15); no longer U1.69B (PG4)
- net EXT_IO_7: now also U1.59B (PF12); no longer U1.65B (PD10)
- net EXT_IO_8: now also U1.64B (PE0); no longer U1.68B (PG5)
- net EXT_IO_9: now also U1.62B (PF11); no longer U1.64B (PE0)
- net LED_RGB_B: now also U1.68B (PG5); no longer U1.57B (PF13)
- net LED_RGB_G: now also U1.69B (PG4); no longer U1.59B (PF12)
- net LED_RGB_R: now also U1.65B (PD10); no longer U1.62B (PF11)
- net ROBOT_SELECT: now also U1.58B (PF3); no longer U1.24B (PB1)
Changed lines of the file:
@@
-	1    0    0    -1
-$EndComp
-$Comp
-L +5V #PWR016
-U 1 1 586DD9D9
-P 5200 6600
-F 0 "#PWR016" H 5200 6690 20  0001 C CNN
-F 1 "+5V" H 5200 6690 30  0000 C CNN
-F 2 "" H 5200 6600 60  0000 C CNN
-F 3 "" H 5200 6600 60  0000 C CNN
-	1    5200 6600
 	1    0    0    -1
 $EndComp
@@
 	1    0    0    -1
 $EndComp
-Text Label 6000 2250 0    50   ~ 0
+Text Label 6000 3950 0    50   ~ 0
 ROBOT_SELECT
 Text Label 4650 5700 0    50   ~ 0
 ROBOT_SELECT
 $Comp
-L GND #PWR017
+L GND #PWR016
 U 1 1 58923511
 P 5250 5800
-F 0 "#PWR017" H 5250 5800 30  0001 C CNN
+F 0 "#PWR016" H 5250 5800 30  0001 C CNN
 F 1 "GND" H 5250 5730 30  0001 C CNN
 F 2 "" H 5250 5800 60  0000 C CNN
@@
 Text Label 2700 3950 0    50   ~ 0
 EXT_IO_4
-Text Label 4700 4550 2    50   ~ 0
+Text Label 6000 4050 0    50   ~ 0
 EXT_IO_6
-Text Label 6000 4450 0    50   ~ 0
+Text Label 6000 4250 0    50   ~ 0
 EXT_IO_8
 Text Label 6000 4350 0    50   ~ 0
 EXT_IO_10
-Text Label 4700 4050 2    50   ~ 0
+Text Label 4700 4550 2    50   ~ 0
 LED_RGB_G
 Text Label 2700 4350 0    50   ~ 0
@@
 Text Label 2700 3850 0    50   ~ 0
 EXT_IO_5
+Text Label 4700 4050 2    50   ~ 0
+EXT_IO_7
+Text Label 6000 4150 0    50   ~ 0
+EXT_IO_9
 Text Label 4700 4350 2    50   ~ 0
-EXT_IO_7
-Text Label 6000 4250 0    50   ~ 0
-EXT_IO_9
-Text Label 6000 4150 0    50   ~ 0
 LED_RGB_R
-Text Label 4700 3950 2    50   ~ 0
+Text Label 6000 4450 0    50   ~ 0
 LED_RGB_B
 $Comp
@@
 (BOOT1)
 $Comp
-L +5V #PWR018
+L +5V #PWR017
 U 1 1 58B898A2
 P 2850 1950
-F 0 "#PWR018" H 2850 2040 20  0001 C CNN
+F 0 "#PWR017" H 2850 2040 20  0001 C CNN
 F 1 "+5V" H 2950 2000 30  0000 C CNN
 F 2 "" H 2850 1950 60  0001 C CNN
@@
 E5V
 $Comp
-L GND #PWR019
+L GND #PWR018
 U 1 1 58BB229F
 P 8700 1950
-F 0 "#PWR019" H 8700 1950 30  0001 C CNN
+F 0 "#PWR018" H 8700 1950 30  0001 C CNN
 F 1 "GND" H 8700 1880 30  0001 C CNN
 F 2 "" H 8700 1950 60  0001 C CNN
@@
 Extension connectors\nnot populated
 $Comp
-L +3.3V #PWR020
+L +3.3V #PWR019
 U 1 1 58BBB142
 P 1800 5650
-F 0 "#PWR020" H 1800 5610 30  0001 C CNN
+F 0 "#PWR019" H 1800 5610 30  0001 C CNN
 F 1 "+3.3V" H 1800 5760 30  0000 C CNN
 F 2 "" H 1800 5650 60  0001 C CNN
@@
 $EndComp
 $Comp
-L +3.3V #PWR021
+L +3.3V #PWR020
 U 1 1 58BBB29E
 P 5250 5600
-F 0 "#PWR021" H 5250 5560 30  0001 C CNN
+F 0 "#PWR020" H 5250 5560 30  0001 C CNN
 F 1 "+3.3V" H 5250 5710 30  0000 C CNN
 F 2 "" H 5250 5600 60  0001 C CNN
@@
 $EndComp
 $Comp
-L +3.3V #PWR022
+L +3.3V #PWR021
 U 1 1 58BBD1A5
 P 10450 5750
-F 0 "#PWR022" H 10450 5710 30  0001 C CNN
+F 0 "#PWR021" H 10450 5710 30  0001 C CNN
 F 1 "+3.3V" H 10450 5860 30  0000 C CNN
 F 2 "" H 10450 5750 60  0001 C CNN
@@
 $EndComp
 $Comp
-L +3.3V #PWR023
+L +3.3V #PWR022
 U 1 1 58BBD2B4
 P 10450 4550
-F 0 "#PWR023" H 10450 4510 30  0001 C CNN
+F 0 "#PWR022" H 10450 4510 30  0001 C CNN
 F 1 "+3.3V" H 10450 4660 30  0000 C CNN
 F 2 "" H 10450 4550 60  0001 C CNN
@@
 $EndComp
 $Comp
-L +3.3V #PWR024
+L +3.3V #PWR023
 U 1 1 58BBD43F
 P 10450 3550
-F 0 "#PWR024" H 10450 3510 30  0001 C CNN
+F 0 "#PWR023" H 10450 3510 30  0001 C CNN
 F 1 "+3.3V" H 10450 3660 30  0000 C CNN
 F 2 "" H 10450 3550 60  0001 C CNN
@@
 $EndComp
 $Comp
-L +3.3V #PWR025
+L +3.3V #PWR024
 U 1 1 58BBD682
 P 8850 750
-F 0 "#PWR025" H 8850 710 30  0001 C CNN
+F 0 "#PWR024" H 8850 710 30  0001 C CNN
 F 1 "+3.3V" H 8850 860 30  0000 C CNN
 F 2 "" H 8850 750 60  0001 C CNN
@@
 $EndComp
 $Comp
-L +5V #PWR026
+L +5V #PWR025
 U 1 1 58BBDB7F
 P 8200 5700
-F 0 "#PWR026" H 8200 5790 20  0001 C CNN
+F 0 "#PWR025" H 8200 5790 20  0001 C CNN
 F 1 "+5V" H 8200 5790 30  0000 C CNN
 F 2 "" H 8200 5700 60  0000 C CNN
@@
 $EndComp
 $Comp
-L +3.3V #PWR027
+L +3.3V #PWR026
 U 1 1 58BBE79F
 P 10150 5500
-F 0 "#PWR027" H 10150 5460 30  0001 C CNN
+F 0 "#PWR026" H 10150 5460 30  0001 C CNN
 F 1 "+3.3V" H 10150 5610 30  0000 C CNN
 F 2 "" H 10150 5500 60  0001 C CNN
@@
 $EndComp
 $Comp
-L +3.3V #PWR028
+L +3.3V #PWR027
 U 1 1 58BBEAB2
 P 2850 1850
-F 0 "#PWR028" H 2850 1810 30  0001 C CNN
+F 0 "#PWR027" H 2850 1810 30  0001 C CNN
 F 1 "+3.3V" H 2950 1900 30  0000 C CNN
 F 2 "" H 2850 1850 60  0001 C CNN
@@
 $EndComp
 $Comp
-L GND #PWR029
+L GND #PWR028
 U 1 1 58BBF197
 P 2700 1450
-F 0 "#PWR029" H 2700 1450 30  0001 C CNN
+F 0 "#PWR028" H 2700 1450 30  0001 C CNN
 F 1 "GND" H 2700 1380 30  0001 C CNN
 F 2 "" H 2700 1450 60  0001 C CNN
@@
 $EndComp
 $Comp
-L GND #PWR030
+L GND #PWR029
 U 1 1 58BBF265
 P 2700 2150
-F 0 "#PWR030" H 2700 2150 30  0001 C CNN
+F 0 "#PWR029" H 2700 2150 30  0001 C CNN
 F 1 "GND" H 2700 2080 30  0001 C CNN
 F 2 "" H 2700 2150 60  0001 C CNN
@@
 	2700 2050 2700 2150
 $Comp
-L GND #PWR031
+L GND #PWR030
 U 1 1 58BC29AE
 P 2700 4050
-F 0 "#PWR031" H 2700 4050 30  0001 C CNN
+F 0 "#PWR030" H 2700 4050 30  0001 C CNN
 F 1 "GND" H 2700 3980 30  0001 C CNN
 F 2 "" H 2700 4050 60  0001 C CNN
@@
 $EndComp
 $Comp
-L GND #PWR032
+L GND #PWR031
 U 1 1 58BC2A7C
 P 1400 3550
-F 0 "#PWR032" H 1400 3550 30  0001 C CNN
+F 0 "#PWR031" H 1400 3550 30  0001 C CNN
 F 1 "GND" H 1400 3480 30  0001 C CNN
 F 2 "" H 1400 3550 60  0001 C CNN
@@
 $EndComp
 $Comp
-L GND #PWR033
+L GND #PWR032
 U 1 1 58BC2B4A
 P 1400 2050
-F 0 "#PWR033" H 1400 2050 30  0001 C CNN
+F 0 "#PWR032" H 1400 2050 30  0001 C CNN
 F 1 "GND" H 1400 1980 30  0001 C CNN
 F 2 "" H 1400 2050 60  0001 C CNN
@@
 $EndComp
 $Comp
-L GND #PWR034
+L GND #PWR033
 U 1 1 58BC2C18
 P 4700 1550
-F 0 "#PWR034" H 4700 1550 30  0001 C CNN
+F 0 "#PWR033" H 4700 1550 30  0001 C CNN
 F 1 "GND" H 4700 1480 30  0001 C CNN
 F 2 "" H 4700 1550 60  0001 C CNN
@@
 $EndComp
 $Comp
-L GND #PWR035
+L GND #PWR034
 U 1 1 58BC2CE6
 P 4700 3050
-F 0 "#PWR035" H 4700 3050 30  0001 C CNN
+F 0 "#PWR034" H 4700 3050 30  0001 C CNN
 F 1 "GND" H 4700 2980 30  0001 C CNN
 F 2 "" H 4700 3050 60  0001 C CNN
@@
 $EndComp
 $Comp
-L GND #PWR036
+L GND #PWR035
 U 1 1 58BC2DB4
 P 4700 4250
-F 0 "#PWR036" H 4700 4250 30  0001 C CNN
+F 0 "#PWR035" H 4700 4250 30  0001 C CNN
 F 1 "GND" H 4700 4180 30  0001 C CNN
 F 2 "" H 4700 4250 60  0001 C CNN
@@
 $EndComp
 $Comp
-L GND #PWR037
+L GND #PWR036
 U 1 1 58BC2E82
 P 6000 3750
-F 0 "#PWR037" H 6000 3750 30  0001 C CNN
+F 0 "#PWR036" H 6000 3750 30  0001 C CNN
 F 1 "GND" H 6000 3680 30  0001 C CNN
 F 2 "" H 6000 3750 60  0001 C CNN
@@
 $EndComp
 $Comp
-L GND #PWR038
+L GND #PWR037
 U 1 1 58BC2F50
 P 6000 2650
-F 0 "#PWR038" H 6000 2650 30  0001 C CNN
+F 0 "#PWR037" H 6000 2650 30  0001 C CNN
 F 1 "GND" H 6000 2580 30  0001 C CNN
 F 2 "" H 6000 2650 60  0001 C CNN
@@
 $EndComp
 $Comp
-L GND #PWR039
+L GND #PWR038
 U 1 1 58BC301E
 P 6000 2050
-F 0 "#PWR039" H 6000 2050 30  0001 C CNN
+F 0 "#PWR038" H 6000 2050 30  0001 C CNN
 F 1 "GND" H 6000 1980 30  0001 C CNN
 F 2 "" H 6000 2050 60  0001 C CNN
@@
 LED_SD
 $Comp
-L GND #PWR040
+L GND #PWR039
 U 1 1 58BCD0B9
 P 1700 7450
-F 0 "#PWR040" H 1700 7450 30  0001 C CNN
+F 0 "#PWR039" H 1700 7450 30  0001 C CNN
 F 1 "GND" H 1700 7380 30  0001 C CNN
 F 2 "" H 1700 7450 60  0001 C CNN
@@
 P 4800 6900
 F 0 "R8" V 4880 6900 50  0000 C CNN
-F 1 "100" V 4800 6900 50  0000 C CNN
+F 1 "0" V 4800 6900 50  0000 C CNN
 F 2 "Resistors_SMD:R_0805" V 4730 6900 50  0001 C CNN
 F 3 "" H 4800 6900 50  0000 C CNN
@@
 NoConn ~ 4700 2150
 NoConn ~ 4700 2250
+$Comp
+L +3.3V #PWR040
+U 1 1 58BD1ED9
+P 5200 6600
+F 0 "#PWR040" H 5200 6560 30  0001 C CNN
+F 1 "+3.3V" H 5200 6710 30  0000 C CNN
+F 2 "" H 5200 6600 60  0001 C CNN
+F 3 "" H 5200 6600 60  0001 C CNN
+	1    5200 6600
+	1    0    0    -1
+$EndComp
 $EndSCHEMATC

Commit message: fix SD PMOS switch pinout
Parts:
- Q1: value Q_PMOS_DGS -> Q_PMOS_GSD; symbol Q_PMOS_DGS -> Q_PMOS_GSD
Connections:
- net +3.3V: now also Q1.2 (S); no longer Q1.1 (D)
- net SD_PWR: now also Q1.1 (G); no longer Q1.2 (G)
- no-connect marks 8 -> 65
Changed lines of the file:
@@
 $EndComp
 $Comp
-L Q_PMOS_DGS Q1
+L Q_PMOS_GSD Q1
 U 1 1 581FC8E7
 P 1700 6000
 F 0 "Q1" H 2000 6050 50  0000 R CNN
-F 1 "Q_PMOS_DGS" H 2350 5950 50  0000 R CNN
+F 1 "Q_PMOS_GSD" H 2350 5950 50  0000 R CNN
 F 2 "TO_SOT_Packages_SMD:SOT-23_Handsoldering" H 1900 6100 50  0001 C CNN
 F 3 "" H 1700 6000 50  0000 C CNN
 	1    1700 6000
-	1    0    0    -1
+	1    0    0    1
 $EndComp
 $Comp
@@
 	1    0    0    -1
 $EndComp
+NoConn ~ 4700 3950
+NoConn ~ 4700 3750
+NoConn ~ 4700 3450
+NoConn ~ 4700 2950
+NoConn ~ 4700 2850
+NoConn ~ 4700 2750
+NoConn ~ 4700 2650
+NoConn ~ 6000 3650
+NoConn ~ 6000 3550
+NoConn ~ 6000 3450
+NoConn ~ 6000 3350
+NoConn ~ 6000 3250
+NoConn ~ 6000 3150
+NoConn ~ 6000 3050
+NoConn ~ 6000 2950
+NoConn ~ 6000 2850
+NoConn ~ 6000 2750
+NoConn ~ 6000 2550
+NoConn ~ 6000 2450
+NoConn ~ 4700 2450
+NoConn ~ 4700 1450
+NoConn ~ 4700 1850
+NoConn ~ 6000 1750
+NoConn ~ 6000 1650
+NoConn ~ 6000 1550
+NoConn ~ 6000 1450
+NoConn ~ 6000 2250
+NoConn ~ 2700 3750
+NoConn ~ 2700 3650
+NoConn ~ 1400 3750
+NoConn ~ 1400 3650
+NoConn ~ 1400 3450
+NoConn ~ 1400 3350
+NoConn ~ 2700 3350
+NoConn ~ 2700 3250
+NoConn ~ 2700 3150
+NoConn ~ 2700 3050
+NoConn ~ 2700 2850
+NoConn ~ 2700 2750
+NoConn ~ 2700 2650
+NoConn ~ 2700 2550
+NoConn ~ 2700 2450
+NoConn ~ 2700 2250
+NoConn ~ 1400 3050
+NoConn ~ 1400 2950
+NoConn ~ 1400 2850
+NoConn ~ 1400 2750
+NoConn ~ 1400 2650
+NoConn ~ 1400 2550
+NoConn ~ 1400 2450
+NoConn ~ 1400 2350
+NoConn ~ 1400 2250
+NoConn ~ 1400 2150
+NoConn ~ 1400 1950
+NoConn ~ 2700 1650
+NoConn ~ 1400 1350
+NoConn ~ 1400 1450
 $EndSCHEMATC
