File: servo.sch (KiCad schematic (older format))
At the start: 19 parts

Commit message: footprint assignment
Parts:
- removed P?: CONN_01X02, symbol CONN_01X02
- added J2: V_SERVO_CONN, Terminal_Blocks:TerminalBlock_Pheonix_MKDS1.5-2pol, symbol Screw_Terminal_1x02
- CONN15, CONN16, CONN17, CONN18, CONN19, CONN20, CONN21, CONN22, CONN23, CONN24, CONN25, CONN26, CONN27, CONN28, CONN29, CONN30: renamed from CONN?; footprint (none) -> Pin_Headers:Pin_Header_Straight_1x03
- R6: renamed from R?; footprint (none) -> Resistors_SMD:R_0603
- U4: renamed from U?; footprint (none) -> Housings_SSOP:TSSOP-28_4.4x9.7mm_Pitch0.65mm
Connections:
- net GND: now also J2.1
- net SERVO_VCC renamed V_SERVO
- net V_SERVO: now also J2.2
- net VCC renamed +3.3V

Commit message: place parts in PCB
Parts:
- R6: footprint Resistors_SMD:R_0603 -> Resistors_SMD:R_0805
Changed lines of the file:
@@
 $EndComp
 $Comp
-L GND #PWR059
+L GND #PWR060
 U 1 1 584D3DB4
 P 1800 2850
-F 0 "#PWR059" H 1800 2850 30  0001 C CNN
+F 0 "#PWR060" H 1800 2850 30  0001 C CNN
 F 1 "GND" H 1800 2780 30  0001 C CNN
 F 2 "" H 1800 2850 60  0000 C CNN
@@
 F 0 "R6" V 1680 1150 50  0000 C CNN
 F 1 "10k" V 1600 1150 50  0000 C CNN
-F 2 "Resistors_SMD:R_0603" V 1530 1150 50  0001 C CNN
+F 2 "Resistors_SMD:R_0805" V 1530 1150 50  0001 C CNN
 F 3 "" H 1600 1150 50  0000 C CNN
 	1    1600 1150
@@
 V_SERVO
 $Comp
-L GND #PWR060
+L GND #PWR061
 U 1 1 584D6571
 P 5050 1400
-F 0 "#PWR060" H 5050 1400 30  0001 C CNN
+F 0 "#PWR061" H 5050 1400 30  0001 C CNN
 F 1 "GND" H 5050 1330 30  0001 C CNN
 F 2 "" H 5050 1400 60  0000 C CNN
@@
 $EndComp
 $Comp
-L GND #PWR061
+L GND #PWR062
 U 1 1 584D65CD
 P 6100 1400
-F 0 "#PWR061" H 6100 1400 30  0001 C CNN
+F 0 "#PWR062" H 6100 1400 30  0001 C CNN
 F 1 "GND" H 6100 1330 30  0001 C CNN
 F 2 "" H 6100 1400 60  0000 C CNN
@@
 $EndComp
 $Comp
-L GND #PWR062
+L GND #PWR063
 U 1 1 584D6617
 P 7150 1400
-F 0 "#PWR062" H 7150 1400 30  0001 C CNN
+F 0 "#PWR063" H 7150 1400 30  0001 C CNN
 F 1 "GND" H 7150 1330 30  0001 C CNN
 F 2 "" H 7150 1400 60  0000 C CNN
@@
 $EndComp
 $Comp
-L GND #PWR063
+L GND #PWR064
 U 1 1 584D6661
 P 8200 1400
-F 0 "#PWR063" H 8200 1400 30  0001 C CNN
+F 0 "#PWR064" H 8200 1400 30  0001 C CNN
 F 1 "GND" H 8200 1330 30  0001 C CNN
 F 2 "" H 8200 1400 60  0000 C CNN
@@
 $EndComp
 $Comp
-L GND #PWR064
+L GND #PWR065
 U 1 1 584D696E
 P 5050 2100
-F 0 "#PWR064" H 5050 2100 30  0001 C CNN
+F 0 "#PWR065" H 5050 2100 30  0001 C CNN
 F 1 "GND" H 5050 2030 30  0001 C CNN
 F 2 "" H 5050 2100 60  0000 C CNN
@@
 $EndComp
 $Comp
-L GND #PWR065
+L GND #PWR066
 U 1 1 584D69B8
 P 6100 2100
-F 0 "#PWR065" H 6100 2100 30  0001 C CNN
+F 0 "#PWR066" H 6100 2100 30  0001 C CNN
 F 1 "GND" H 6100 2030 30  0001 C CNN
 F 2 "" H 6100 2100 60  0000 C CNN
@@
 $EndComp
 $Comp
-L GND #PWR066
+L GND #PWR067
 U 1 1 584D6A02
 P 7150 2100
-F 0 "#PWR066" H 7150 2100 30  0001 C CNN
+F 0 "#PWR067" H 7150 2100 30  0001 C CNN
 F 1 "GND" H 7150 2030 30  0001 C CNN
 F 2 "" H 7150 2100 60  0000 C CNN
@@
 $EndComp
 $Comp
-L GND #PWR067
+L GND #PWR068
 U 1 1 584D6A4C
 P 8200 2100
-F 0 "#PWR067" H 8200 2100 30  0001 C CNN
+F 0 "#PWR068" H 8200 2100 30  0001 C CNN
 F 1 "GND" H 8200 2030 30  0001 C CNN
 F 2 "" H 8200 2100 60  0000 C CNN
@@
 $EndComp
 $Comp
-L GND #PWR068
+L GND #PWR069
 U 1 1 584D6A96
 P 5050 2850
-F 0 "#PWR068" H 5050 2850 30  0001 C CNN
+F 0 "#PWR069" H 5050 2850 30  0001 C CNN
 F 1 "GND" H 5050 2780 30  0001 C CNN
 F 2 "" H 5050 2850 60  0000 C CNN
@@
 $EndComp
 $Comp
-L GND #PWR069
+L GND #PWR070
 U 1 1 584D6B20
 P 6100 2850
-F 0 "#PWR069" H 6100 2850 30  0001 C CNN
+F 0 "#PWR070" H 6100 2850 30  0001 C CNN
 F 1 "GND" H 6100 2780 30  0001 C CNN
 F 2 "" H 6100 2850 60  0000 C CNN
@@
 $EndComp
 $Comp
-L GND #PWR070
+L GND #PWR071
 U 1 1 584D6B6A
 P 7150 2850
-F 0 "#PWR070" H 7150 2850 30  0001 C CNN
+F 0 "#PWR071" H 7150 2850 30  0001 C CNN
 F 1 "GND" H 7150 2780 30  0001 C CNN
 F 2 "" H 7150 2850 60  0000 C CNN
@@
 $EndComp
 $Comp
-L GND #PWR071
+L GND #PWR072
 U 1 1 584D6BB4
 P 8200 2850
-F 0 "#PWR071" H 8200 2850 30  0001 C CNN
+F 0 "#PWR072" H 8200 2850 30  0001 C CNN
 F 1 "GND" H 8200 2780 30  0001 C CNN
 F 2 "" H 8200 2850 60  0000 C CNN
@@
 $EndComp
 $Comp
-L GND #PWR072
+L GND #PWR073
 U 1 1 584D6BFE
 P 5050 3600
-F 0 "#PWR072" H 5050 3600 30  0001 C CNN
+F 0 "#PWR073" H 5050 3600 30  0001 C CNN
 F 1 "GND" H 5050 3530 30  0001 C CNN
 F 2 "" H 5050 3600 60  0000 C CNN
@@
 $EndComp
 $Comp
-L GND #PWR073
+L GND #PWR074
 U 1 1 584D6C48
 P 6100 3600
-F 0 "#PWR073" H 6100 3600 30  0001 C CNN
+F 0 "#PWR074" H 6100 3600 30  0001 C CNN
 F 1 "GND" H 6100 3530 30  0001 C CNN
 F 2 "" H 6100 3600 60  0000 C CNN
@@
 $EndComp
 $Comp
-L GND #PWR074
+L GND #PWR075
 U 1 1 584D6C92
 P 7150 3600
-F 0 "#PWR074" H 7150 3600 30  0001 C CNN
+F 0 "#PWR075" H 7150 3600 30  0001 C CNN
 F 1 "GND" H 7150 3530 30  0001 C CNN
 F 2 "" H 7150 3600 60  0000 C CNN
@@
 $EndComp
 $Comp
-L GND #PWR075
+L GND #PWR076
 U 1 1 584D6CDC
 P 8200 3600
-F 0 "#PWR075" H 8200 3600 30  0001 C CNN
+F 0 "#PWR076" H 8200 3600 30  0001 C CNN
 F 1 "GND" H 8200 3530 30  0001 C CNN
 F 2 "" H 8200 3600 60  0000 C CNN
@@
 V_SERVO
 $Comp
-L GND #PWR076
+L GND #PWR077
 U 1 1 585AE6B7
 P 3900 1450
-F 0 "#PWR076" H 3900 1450 30  0001 C CNN
+F 0 "#PWR077" H 3900 1450 30  0001 C CNN
 F 1 "GND" H 3900 1380 30  0001 C CNN
 F 2 "" H 3900 1450 60  0000 C CNN
@@
 $EndComp
 $Comp
-L +3.3V #PWR077
+L +3.3V #PWR078
 U 1 1 58BBA49C
 P 1600 950
-F 0 "#PWR077" H 1600 910 30  0001 C CNN
+F 0 "#PWR078" H 1600 910 30  0001 C CNN
 F 1 "+3.3V" H 1600 1060 30  0000 C CNN
 F 2 "" H 1600 950 60  0001 C CNN

Commit message: PCB routing
Connections:
- net GND: now also J2.2; no longer J2.1
- net V_SERVO: now also J2.1; no longer J2.2
Changed lines of the file:
@@
 Text Label 8200 2000 2    60   ~ 0
 V_SERVO
-Text Label 3900 1250 2    60   ~ 0
+Text Label 3450 1450 0    60   ~ 0
 V_SERVO
 $Comp
 L GND #PWR077
 U 1 1 585AE6B7
-P 3900 1450
-F 0 "#PWR077" H 3900 1450 30  0001 C CNN
-F 1 "GND" H 3900 1380 30  0001 C CNN
-F 2 "" H 3900 1450 60  0000 C CNN
-F 3 "" H 3900 1450 60  0000 C CNN
-	1    3900 1450
+P 3900 1250
+F 0 "#PWR077" H 3900 1250 30  0001 C CNN
+F 1 "GND" H 3900 1180 30  0001 C CNN
+F 2 "" H 3900 1250 60  0000 C CNN
+F 3 "" H 3900 1250 60  0000 C CNN
+	1    3900 1250
 	1    0    0    -1
 $EndComp
@@
 	1600 950  1600 1000
 Connection ~ 1600 1000
+Wire Wire Line
+	3450 1450 3900 1450
 $EndSCHEMATC
